File: kicad/bloxorz.kicad_pcb (KiCad board)
At the start: 2 copper layers, 63.8 x 47.2 mm, 39 parts, among them CON1 vectrex-edge-connector, J1 PICKIT, J2 RX, J3 TX, J4 DIN_5, J5 GND, SW1 SW_DPST, U1 PIC16F18323, U2 SST39SF040-TSOP, U3 6N135, Y1 8 MHz oscillator

Commit message: PCB rev 3
Parts:
- removed J2: RX, Pin_Headers:Pin_Header_Straight_1x01_Pitch2.54mm
- removed J3: TX, Pin_Headers:Pin_Header_Straight_1x01_Pitch2.54mm
- removed R10, R11, R14, R15, R16, R3, R4, R5, R6, R7, R8, R9: 0, Resistors_SMD:R_0603_HandSoldering
- removed R12: 10k, Resistors_SMD:R_0603_HandSoldering
- C1, C2, C3: footprint Capacitors_SMD:C_0603_HandSoldering -> Capacitors_SMD:C_0805_HandSoldering
- R1, R2: value 0 -> 10k; footprint Resistors_SMD:R_0603_HandSoldering -> Resistors_SMD:R_0805_HandSoldering
- R13: footprint Resistors_SMD:R_1206_HandSoldering -> Resistors_SMD:R_0805_HandSoldering
- R17: footprint Resistors_SMD:R_0603_HandSoldering -> Resistors_SMD:R_0805_HandSoldering
- U3: footprint Housings_DIP:DIP-8_W7.62mm_SMD -> Housings_DIP:DIP-8_W8.89mm_SMDSocket_LongPads
- moved R1 28.1 mm to (159.1, 79.0), turned to 90 degrees
- moved U2 3.71 mm to (156.2, 56.6)
- moved R19 3.07 mm to (138.9, 85.0)
- moved R18 3.05 mm to (138.9, 82.0)
- moved C3 2.82 mm to (146.8, 54.5), turned to 270 degrees
- moved R17 2.20 mm to (132.6, 83.8)
- moved U3 1.04 mm to (124.8, 81.7)
- moved hole4 1.00 mm to (134.5, 52.3)
- moved hole5 1.00 mm to (134.5, 76.2)
- moved hole3 0.20 mm to (163.0, 84.1)
- moved hole2 0.10 mm to (163.0, 64.2)
- moved hole1 0.06 mm to (163.0, 44.4)
Connections:
- net Net-(CON1-Pad17) renamed A0
- net Net-(CON1-Pad18) renamed D7
- net Net-(CON1-Pad23) renamed D2
- net Net-(CON1-Pad6) renamed A8
- CON1 pad 10: Net-(CON1-Pad10) -> A11
- CON1 pad 11: Net-(CON1-Pad11) -> A3
- CON1 pad 13: Net-(CON1-Pad13) -> A2
- CON1 pad 14: Net-(CON1-Pad14) -> A10
- CON1 pad 15: Net-(CON1-Pad15) -> A1
- CON1 pad 19: Net-(CON1-Pad19) -> D0
- CON1 pad 20: Net-(CON1-Pad20) -> D6
- CON1 pad 21: Net-(CON1-Pad21) -> D1
- CON1 pad 22: Net-(CON1-Pad22) -> D5
- CON1 pad 24: Net-(CON1-Pad24) -> D4
- CON1 pad 26: Net-(CON1-Pad26) -> D3
- CON1 pad 29: Net-(CON1-Pad29) -> A12
- CON1 pad 3: Net-(CON1-Pad3) -> A7
- CON1 pad 31: Net-(CON1-Pad31) -> A13
- CON1 pad 33: Net-(CON1-Pad33) -> A14
- CON1 pad 5: Net-(CON1-Pad5) -> A6
- CON1 pad 7: Net-(CON1-Pad7) -> A5
- CON1 pad 8: Net-(CON1-Pad8) -> A9
- CON1 pad 9: Net-(CON1-Pad9) -> A4
- J1 pad 4: Net-(J1-Pad4) -> V-CE
- J1 pad 5: Net-(J1-Pad5) -> A18
- R1 pad 1: GND -> +5V
- R1 pad 2: Net-(R1-Pad2) -> V-PB6
- R2 pad 1: GND -> +5V
- R2 pad 2: Net-(R2-Pad2) -> V-HALT
- SW1 pad 1: Net-(R12-Pad2) -> Net-(J1-Pad1)
- SW1 pad 3: GND -> Net-(J1-Pad1)
- U1 pad 10: Net-(R8-Pad2) -> A15
- U1 pad 11: Net-(R12-Pad2) -> A16
- U1 pad 12: Net-(J1-Pad5) -> A18
- U1 pad 13: Net-(J1-Pad4) -> V-CE
- U1 pad 5: Net-(J3-Pad1) -> Net-(U1-Pad5)
- U1 pad 7: Net-(R5-Pad2) -> V-PB6
- U1 pad 8: Net-(R6-Pad2) -> V-OE
- U1 pad 9: Net-(R7-Pad2) -> A17
- U2 pad 1: Net-(CON1-Pad10) -> A7
- U2 pad 10: Net-(R1-Pad2) -> A16
- U2 pad 11: Net-(R4-Pad1) -> A15
- U2 pad 12: Net-(CON1-Pad29) -> A4
- U2 pad 13: Net-(CON1-Pad3) -> A11
- U2 pad 14: Net-(CON1-Pad5) -> A3
- U2 pad 15: Net-(CON1-Pad7) -> A2
- U2 pad 16: Net-(CON1-Pad9) -> A10
- U2 pad 17: Net-(CON1-Pad11) -> A14
- U2 pad 18: Net-(CON1-Pad13) -> A13
- U2 pad 19: Net-(CON1-Pad15) -> A12
- U2 pad 2: Net-(CON1-Pad8) -> A6
- U2 pad 21: Net-(CON1-Pad19) -> D3
- U2 pad 22: Net-(CON1-Pad21) -> D4
- U2 pad 24: Net-(R11-Pad1) -> GND
- U2 pad 25: Net-(CON1-Pad26) -> D5
- U2 pad 26: Net-(CON1-Pad24) -> D1
- U2 pad 27: Net-(CON1-Pad22) -> D6
- U2 pad 28: Net-(CON1-Pad20) -> D0
- U2 pad 30: (no net) -> Net-(U1-Pad5)
- U2 pad 31: Net-(CON1-Pad14) -> A1
- U2 pad 32: Net-(R10-Pad1) -> V-OE
- U2 pad 4: Net-(CON1-Pad31) -> A5
- U2 pad 5: Net-(CON1-Pad33) -> A9
- U2 pad 6: Net-(R2-Pad2) -> A17
- U2 pad 7: Net-(R9-Pad1) -> V-RW
- U2 pad 9: Net-(R3-Pad2) -> A18
Routing:
- net GND: track 126.5 -> 195.8 mm, vias 10 -> 6
- net Net-(CON1-Pad33): track 49.4 -> 0.00 mm, vias 3 -> 0
- net Net-(CON1-Pad31): track 45.9 -> 0.00 mm, vias 3 -> 0
- net Net-(R12-Pad2): track 42.7 -> 0.00 mm, vias 1 -> 0
- net Net-(U1-Pad5): track 0.00 -> 41.8 mm
- net Net-(CON1-Pad29): track 41.7 -> 0.00 mm, vias 3 -> 0
- net A14: track 0.00 -> 37.0 mm, vias 0 -> 1
- net A18: track 0.00 -> 36.4 mm, vias 0 -> 2
- net Net-(CON1-Pad26): track 35.8 -> 0.00 mm, vias 2 -> 0
- net Net-(J1-Pad5): track 33.7 -> 0.00 mm, vias 1 -> 0
- net Net-(R1-Pad2): track 33.0 -> 0.00 mm, vias 2 -> 0
- net A2: track 0.00 -> 33.0 mm, vias 0 -> 1
- net A10: track 0.00 -> 32.9 mm, vias 0 -> 2
- net Net-(CON1-Pad3): track 32.7 -> 0.00 mm, vias 1 -> 0
- net Net-(CON1-Pad5): track 31.8 -> 0.00 mm, vias 1 -> 0
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Other:
- net class Default: clearance 0.1524 -> 0.2032; trace_width 0.2032 -> 0.254; via_dia 0.6858 -> 0.762; via_drill 0.3302 -> 0.508
- rule trace_clearance: 0.1524 -> 0.2032
- rule trace_min: 0.2032 -> 0.1524
- rule via_min_drill: 0.3302 -> 0.508
- rule via_min_size: 0.6858 -> 0.762
- board text added: "Bloxorz - PCB rev 3"
- board text removed: "Bloxorz - PCB rev 2"

Commit message: rev 4
Parts:
- added REF***: WEEE-Logo_4.2x6mm_SilkScreen, Symbols:WEEE-Logo_4.2x6mm_SilkScreen, F.Cu at (150.9, 63.6)
- added REF***: OSHW-Logo2_9.8x8mm_SilkScreen, Symbols:OSHW-Logo2_9.8x8mm_SilkScreen, F.Cu at (162.6, 72.3)
- added REF***: CE-Logo_8.5x6mm_SilkScreen, Symbols:CE-Logo_8.5x6mm_SilkScreen, F.Cu at (142.6, 61.7)
- R13: footprint Resistors_SMD:R_0805_HandSoldering -> Resistors_SMD:R_1206_HandSoldering
- moved hole4 1.50 mm to (133.0, 52.3)
- moved hole5 1.50 mm to (133.0, 76.2)
- moved U3 0.92 mm to (124.3, 82.4)
- moved hole1 0.20 mm to (163.2, 44.4)
- moved hole2 0.20 mm to (163.2, 64.2)
- moved hole3 0.20 mm to (163.2, 84.1)
Routing:
- net Net-(U1-Pad5): track 41.8 -> 28.3 mm
- net Net-(D1-Pad2): track 24.6 -> 17.8 mm
- net GND: track 195.8 -> 194.3 mm
- net Net-(R19-Pad2): track 46.6 -> 45.4 mm
- net +5V: track 141.5 -> 142.6 mm
- net Net-(D1-Pad1): track 38.2 -> 38.9 mm
Other:
- board text added: "Bloxorz - rev 4"
- board text added: "Made in Germany"
- board text removed: "Bloxorz - PCB rev 3"
