File: kicad/bloxorz.kicad_pcb (KiCad board)
At the start: 2 copper layers, 63.8 x 47.2 mm, 27 parts, among them CON1 vectrex-edge-connector, J1 PICKIT, J4 DIN_5, J5 GND, SW1 SW_DPST, U1 PIC16F18323, U2 SST39SF040-TSOP, U3 6N135, Y1 8 MHz oscillator

Commit message: cartridge bus and PB6 on PIO, PIC fixes (A17 pin, MIDI receive), game PB6 register and timing fixes, games menu, flash scripts and protocol docs
Other:
- net class Default removed
