File: kicad/bloxorz.sch (KiCad schematic (older format))
At the start: 19 parts, among them CON1 vectrex-edge-connector, J1 PICKIT, J2 RX, J4 DIN_5, J5 GND, SW1 SW_DPST, U1 PIC16F18323, U3 6N135, Y1 8 MHz oscillator

Commit message: PCB rev 3
Parts:
- removed J2: RX, Pin_Headers:Pin_Header_Straight_1x01_Pitch2.54mm, symbol CONN_01X01
- added R2: 10k, Resistors_SMD:R_0805_HandSoldering, symbol R
- C1, C2, C3: footprint Capacitors_SMD:C_0603_HandSoldering -> Capacitors_SMD:C_0805_HandSoldering
- R1: renamed from R?; footprint Resistors_SMD:R_0603_HandSoldering -> Resistors_SMD:R_0805_HandSoldering
- R13: footprint Resistors_SMD:R_1206_HandSoldering -> Resistors_SMD:R_0805_HandSoldering
- R17: footprint Resistors_SMD:R_0603_HandSoldering -> Resistors_SMD:R_0805_HandSoldering
- U3: footprint Housings_DIP:DIP-8_W7.62mm_SMD -> Housings_DIP:DIP-8_W8.89mm_SMDSocket_LongPads
- gave numbers to parts that had none: 1
Connections:
- net +5V: now also R2.1
- net V-HALT: now also R2.2
- net V-OE: now also U1.8 (RC2); no longer U1.11 (RA2)
- net V-PB6: now also U1.7 (RC3); no longer J1.5 (P5), U1.12 (RA1/ICSPCLK)
- net A15: now reaches U1.10 (RC0)
- net A15: now also U2.11 (A15); no longer U2.9 (A18)
- net A16: now reaches U2.10 (A16)
- net A16: now also U1.11 (RA2); no longer U1.8 (RC2)
- net A17: now reaches U1.9 (RC1), U2.6 (A17)
- net A11: now reaches CON1.10 (A11)
- net A11: now also U2.13 (A7); no longer U2.1 (A11)
- net A14: now reaches U2.17 (A3)
- net A14: now also CON1.33 (A14); no longer CON1.11 (A3)
- net A13: now reaches U2.18 (A2)
- net A13: now also CON1.31 (A13); no longer CON1.13 (A2)
- net A1: now reaches U2.31 (A10)
- net A1: now also CON1.15 (A1); no longer CON1.14 (A10)
- net A12: now reaches U2.19 (A1)
- net A12: now also CON1.29 (A12); no longer CON1.15 (A1)
- net A0: now reaches CON1.17 (A0), U2.20 (A0)
- net D7: now reaches CON1.18 (D7), U2.29 (D7)
- net D0: now reaches CON1.19 (D0)
- net D0: now also U2.28 (D6); no longer U2.21 (D0)
- net D6: now reaches CON1.20 (D6)
- net D6: now also U2.27 (D5); no longer U2.28 (D6)
- net D1: now reaches CON1.21 (D1)
- net D1: now also U2.26 (D4); no longer U2.22 (D1)
- net D5: now reaches CON1.22 (D5)
- net D5: now also U2.25 (D3); no longer U2.27 (D5)
- net D2: now reaches CON1.23 (D2), U2.23 (D2)
- net D4: now reaches CON1.24 (D4)
- net D4: now also U2.22 (D1); no longer U2.26 (D4)
- net D3: now reaches CON1.26 (D3)
- net D3: now also U2.21 (D0); no longer U2.25 (D3)
- net A4: now reaches U2.12 (A12)
- net A4: now also CON1.9 (A4); no longer CON1.29 (A12)
- net A7: now reaches CON1.3 (A7)
- net A7: now also U2.1 (A11); no longer U2.13 (A7)
- net A5: now reaches U2.4 (A13)
- net A5: now also CON1.7 (A5); no longer CON1.31 (A13)
- net A9: now reaches U2.5 (A14)
- net A9: now also CON1.8 (A9); no longer CON1.33 (A14)
- net A3: now reaches U2.14 (A6)
- net A3: now also CON1.11 (A3); no longer CON1.5 (A6)
- net A8: now reaches CON1.6 (A8), U2.3 (A8)
- net A2: now reaches U2.15 (A5)
- net A2: now also CON1.13 (A2); no longer CON1.7 (A5)
- net A6: now reaches U2.2 (A9)
- net A6: now also CON1.5 (A6); no longer CON1.8 (A9)
- net A10: now reaches U2.16 (A4)
- net A10: now also CON1.14 (A10); no longer CON1.9 (A4)
- new net A18: J1.5 (P5), U1.12 (RA1/ICSPCLK), U2.9 (A18)
Other:
- moved on the sheet: C1, C2, C3, CON1, D1, J1, J4, J5, R1, R13, R17, R18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

Commit message: rev 4
Parts:
- R13: footprint Resistors_SMD:R_0805_HandSoldering -> Resistors_SMD:R_1206_HandSoldering
Other:
- moved on the sheet: C1, C2, C3, CON1, D1, J1, J4, J5, R1, R13, R17, R18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
